File: nkns1dvt.sch (KiCad schematic (older format))
At the start: 70 parts, among them J1 MJ-4PP-9, J2 SERIAL_LED, SW1 SW_RESET, SW10 SW_PUSH, SW11 SW_PUSH, SW12 SW_PUSH, SW13 SW_PUSH, SW14 SW_PUSH, SW15 SW_PUSH, SW16 SW_PUSH, SW17 SW_PUSH, SW18 SW_PUSH, SW19 SW_PUSH, SW2 SW_PUSH, SW20 SW_PUSH, SW21 SW_PUSH, SW22 SW_PUSH, SW23 SW_PUSH, SW24 SW_PUSH, SW25 SW_PUSH, SW26 SW_PUSH, SW27 SW_PUSH, SW28 SW_PUSH, SW29 SW_PUSH, SW3 SW_PUSH, SW30 SW_PUSH, SW31 SW_PUSH, SW32 SW_PUSH, SW33 SW_PUSH, SW34 SW_PUSH, SW4 SW_PUSH, SW5 SW_PUSH, SW6 SW_PUSH, SW7 SW_PUSH, SW8 SW_PUSH, SW9 SW_PUSH, U1 ProMicro

Commit message: Change diode footprints
Parts:
- D1, D10, D11, D12, D13, D14, D15, D16, D17, D18, D19, D2, D20, D21, D22, D23, D24, D25, D26, D27, D28, D29, D3, D30, D31, D32, D33, D4, D5, D6, D7, D8, D9: footprint kbd:D3_TH -> kbd:D3_TH_SMD
Changed lines of the file:
@@
 F 0 "D3" V 3996 1470 50  0000 R CNN
 F 1 "D" V 3905 1470 50  0000 R CNN
-F 2 "kbd:D3_TH" H 3950 1550 50  0001 C CNN
+F 2 "kbd:D3_TH_SMD" H 3950 1550 50  0001 C CNN
 F 3 "~" H 3950 1550 50  0001 C CNN
 	1    3950 1550
@@
 F 0 "D2" V 2846 1470 50  0000 R CNN
 F 1 "D" V 2755 1470 50  0000 R CNN
-F 2 "kbd:D3_TH" H 2800 1550 50  0001 C CNN
+F 2 "kbd:D3_TH_SMD" H 2800 1550 50  0001 C CNN
 F 3 "~" H 2800 1550 50  0001 C CNN
 	1    2800 1550
@@
 F 0 "D1" V 1696 1470 50  0000 R CNN
 F 1 "D" V 1605 1470 50  0000 R CNN
-F 2 "kbd:D3_TH" H 1650 1550 50  0001 C CNN
+F 2 "kbd:D3_TH_SMD" H 1650 1550 50  0001 C CNN
 F 3 "~" H 1650 1550 50  0001 C CNN
 	1    1650 1550
@@
 F 0 "D7" V 1696 2470 50  0000 R CNN
 F 1 "D" V 1605 2470 50  0000 R CNN
-F 2 "kbd:D3_TH" H 1650 2550 50  0001 C CNN
+F 2 "kbd:D3_TH_SMD" H 1650 2550 50  0001 C CNN
 F 3 "~" H 1650 2550 50  0001 C CNN
 	1    1650 2550
@@
 F 0 "D8" V 2846 2470 50  0000 R CNN
 F 1 "D" V 2755 2470 50  0000 R CNN
-F 2 "kbd:D3_TH" H 2800 2550 50  0001 C CNN
+F 2 "kbd:D3_TH_SMD" H 2800 2550 50  0001 C CNN
 F 3 "~" H 2800 2550 50  0001 C CNN
 	1    2800 2550
@@
 F 0 "D9" V 3996 2470 50  0000 R CNN
 F 1 "D" V 3905 2470 50  0000 R CNN
-F 2 "kbd:D3_TH" H 3950 2550 50  0001 C CNN
+F 2 "kbd:D3_TH_SMD" H 3950 2550 50  0001 C CNN
 F 3 "~" H 3950 2550 50  0001 C CNN
 	1    3950 2550
@@
 F 0 "D15" V 3996 3470 50  0000 R CNN
 F 1 "D" V 3905 3470 50  0000 R CNN
-F 2 "kbd:D3_TH" H 3950 3550 50  0001 C CNN
+F 2 "kbd:D3_TH_SMD" H 3950 3550 50  0001 C CNN
 F 3 "~" H 3950 3550 50  0001 C CNN
 	1    3950 3550
@@
 F 0 "D14" V 2846 3470 50  0000 R CNN
 F 1 "D" V 2755 3470 50  0000 R CNN
-F 2 "kbd:D3_TH" H 2800 3550 50  0001 C CNN
+F 2 "kbd:D3_TH_SMD" H 2800 3550 50  0001 C CNN
 F 3 "~" H 2800 3550 50  0001 C CNN
 	1    2800 3550
@@
 F 0 "D13" V 1696 3470 50  0000 R CNN
 F 1 "D" V 1605 3470 50  0000 R CNN
-F 2 "kbd:D3_TH" H 1650 3550 50  0001 C CNN
+F 2 "kbd:D3_TH_SMD" H 1650 3550 50  0001 C CNN
 F 3 "~" H 1650 3550 50  0001 C CNN
 	1    1650 3550
@@
 F 0 "D19" V 1696 4520 50  0000 R CNN
 F 1 "D" V 1605 4520 50  0000 R CNN
-F 2 "kbd:D3_TH" H 1650 4600 50  0001 C CNN
+F 2 "kbd:D3_TH_SMD" H 1650 4600 50  0001 C CNN
 F 3 "~" H 1650 4600 50  0001 C CNN
 	1    1650 4600
@@
 F 0 "D20" V 2846 4520 50  0000 R CNN
 F 1 "D" V 2755 4520 50  0000 R CNN
-F 2 "kbd:D3_TH" H 2800 4600 50  0001 C CNN
+F 2 "kbd:D3_TH_SMD" H 2800 4600 50  0001 C CNN
 F 3 "~" H 2800 4600 50  0001 C CNN
 	1    2800 4600
@@
 F 0 "D21" V 3996 4520 50  0000 R CNN
 F 1 "D" V 3905 4520 50  0000 R CNN
-F 2 "kbd:D3_TH" H 3950 4600 50  0001 C CNN
+F 2 "kbd:D3_TH_SMD" H 3950 4600 50  0001 C CNN
 F 3 "~" H 3950 4600 50  0001 C CNN
 	1    3950 4600
@@
 F 0 "D28" V 3996 5570 50  0000 R CNN
 F 1 "D" V 3905 5570 50  0000 R CNN
-F 2 "kbd:D3_TH" H 3950 5650 50  0001 C CNN
+F 2 "kbd:D3_TH_SMD" H 3950 5650 50  0001 C CNN
 F 3 "~" H 3950 5650 50  0001 C CNN
 	1    3950 5650
@@
 F 0 "D27" V 2846 5570 50  0000 R CNN
 F 1 "D" V 2755 5570 50  0000 R CNN
-F 2 "kbd:D3_TH" H 2800 5650 50  0001 C CNN
+F 2 "kbd:D3_TH_SMD" H 2800 5650 50  0001 C CNN
 F 3 "~" H 2800 5650 50  0001 C CNN
 	1    2800 5650
@@
 F 0 "D26" V 1696 5570 50  0000 R CNN
 F 1 "D" V 1605 5570 50  0000 R CNN
-F 2 "kbd:D3_TH" H 1650 5650 50  0001 C CNN
+F 2 "kbd:D3_TH_SMD" H 1650 5650 50  0001 C CNN
 F 3 "~" H 1650 5650 50  0001 C CNN
 	1    1650 5650
@@
 F 0 "D29" V 5146 5570 50  0000 R CNN
 F 1 "D" V 5055 5570 50  0000 R CNN
-F 2 "kbd:D3_TH" H 5100 5650 50  0001 C CNN
+F 2 "kbd:D3_TH_SMD" H 5100 5650 50  0001 C CNN
 F 3 "~" H 5100 5650 50  0001 C CNN
 	1    5100 5650
@@
 F 0 "D30" V 6296 5570 50  0000 R CNN
 F 1 "D" V 6205 5570 50  0000 R CNN
-F 2 "kbd:D3_TH" H 6250 5650 50  0001 C CNN
+F 2 "kbd:D3_TH_SMD" H 6250 5650 50  0001 C CNN
 F 3 "~" H 6250 5650 50  0001 C CNN
 	1    6250 5650
@@
 F 0 "D31" V 7446 5570 50  0000 R CNN
 F 1 "D" V 7355 5570 50  0000 R CNN
-F 2 "kbd:D3_TH" H 7400 5650 50  0001 C CNN
+F 2 "kbd:D3_TH_SMD" H 7400 5650 50  0001 C CNN
 F 3 "~" H 7400 5650 50  0001 C CNN
 	1    7400 5650
@@
 F 0 "D32" V 8596 5570 50  0000 R CNN
 F 1 "D" V 8505 5570 50  0000 R CNN
-F 2 "kbd:D3_TH" H 8550 5650 50  0001 C CNN
+F 2 "kbd:D3_TH_SMD" H 8550 5650 50  0001 C CNN
 F 3 "~" H 8550 5650 50  0001 C CNN
 	1    8550 5650
@@
 F 0 "D33" V 9746 5570 50  0000 R CNN
 F 1 "D" V 9655 5570 50  0000 R CNN
-F 2 "kbd:D3_TH" H 9700 5650 50  0001 C CNN
+F 2 "kbd:D3_TH_SMD" H 9700 5650 50  0001 C CNN
 F 3 "~" H 9700 5650 50  0001 C CNN
 	1    9700 5650
@@
 F 0 "D25" V 8596 4520 50  0000 R CNN
 F 1 "D" V 8505 4520 50  0000 R CNN
-F 2 "kbd:D3_TH" H 8550 4600 50  0001 C CNN
+F 2 "kbd:D3_TH_SMD" H 8550 4600 50  0001 C CNN
 F 3 "~" H 8550 4600 50  0001 C CNN
 	1    8550 4600
@@
 F 0 "D24" V 7446 4520 50  0000 R CNN
 F 1 "D" V 7355 4520 50  0000 R CNN
-F 2 "kbd:D3_TH" H 7400 4600 50  0001 C CNN
+F 2 "kbd:D3_TH_SMD" H 7400 4600 50  0001 C CNN
 F 3 "~" H 7400 4600 50  0001 C CNN
 	1    7400 4600
@@
 F 0 "D23" V 6296 4520 50  0000 R CNN
 F 1 "D" V 6205 4520 50  0000 R CNN
-F 2 "kbd:D3_TH" H 6250 4600 50  0001 C CNN
+F 2 "kbd:D3_TH_SMD" H 6250 4600 50  0001 C CNN
 F 3 "~" H 6250 4600 50  0001 C CNN
 	1    6250 4600
@@
 F 0 "D22" V 5146 4520 50  0000 R CNN
 F 1 "D" V 5055 4520 50  0000 R CNN
-F 2 "kbd:D3_TH" H 5100 4600 50  0001 C CNN
+F 2 "kbd:D3_TH_SMD" H 5100 4600 50  0001 C CNN
 F 3 "~" H 5100 4600 50  0001 C CNN
 	1    5100 4600
@@
 F 0 "D16" V 5146 3470 50  0000 R CNN
 F 1 "D" V 5055 3470 50  0000 R CNN
-F 2 "kbd:D3_TH" H 5100 3550 50  0001 C CNN
+F 2 "kbd:D3_TH_SMD" H 5100 3550 50  0001 C CNN
 F 3 "~" H 5100 3550 50  0001 C CNN
 	1    5100 3550
@@
 F 0 "D17" V 6296 3470 50  0000 R CNN
 F 1 "D" V 6205 3470 50  0000 R CNN
-F 2 "kbd:D3_TH" H 6250 3550 50  0001 C CNN
+F 2 "kbd:D3_TH_SMD" H 6250 3550 50  0001 C CNN
 F 3 "~" H 6250 3550 50  0001 C CNN
 	1    6250 3550
@@
 F 0 "D11" V 6296 2470 50  0000 R CNN
 F 1 "D" V 6205 2470 50  0000 R CNN
-F 2 "kbd:D3_TH" H 6250 2550 50  0001 C CNN
+F 2 "kbd:D3_TH_SMD" H 6250 2550 50  0001 C CNN
 F 3 "~" H 6250 2550 50  0001 C CNN
 	1    6250 2550
@@
 F 0 "D10" V 5146 2470 50  0000 R CNN
 F 1 "D" V 5055 2470 50  0000 R CNN
-F 2 "kbd:D3_TH" H 5100 2550 50  0001 C CNN
+F 2 "kbd:D3_TH_SMD" H 5100 2550 50  0001 C CNN
 F 3 "~" H 5100 2550 50  0001 C CNN
 	1    5100 2550
@@
 F 0 "D4" V 5146 1470 50  0000 R CNN
 F 1 "D" V 5055 1470 50  0000 R CNN
-F 2 "kbd:D3_TH" H 5100 1550 50  0001 C CNN
+F 2 "kbd:D3_TH_SMD" H 5100 1550 50  0001 C CNN
 F 3 "~" H 5100 1550 50  0001 C CNN
 	1    5100 1550
@@
 F 0 "D5" V 6296 1470 50  0000 R CNN
 F 1 "D" V 6205 1470 50  0000 R CNN
-F 2 "kbd:D3_TH" H 6250 1550 50  0001 C CNN
+F 2 "kbd:D3_TH_SMD" H 6250 1550 50  0001 C CNN
 F 3 "~" H 6250 1550 50  0001 C CNN
 	1    6250 1550
@@
 F 0 "D18" V 7446 3470 50  0000 R CNN
 F 1 "D" V 7355 3470 50  0000 R CNN
-F 2 "kbd:D3_TH" H 7400 3550 50  0001 C CNN
+F 2 "kbd:D3_TH_SMD" H 7400 3550 50  0001 C CNN
 F 3 "~" H 7400 3550 50  0001 C CNN
 	1    7400 3550
@@
 F 0 "D12" V 7446 2470 50  0000 R CNN
 F 1 "D" V 7355 2470 50  0000 R CNN
-F 2 "kbd:D3_TH" H 7400 2550 50  0001 C CNN
+F 2 "kbd:D3_TH_SMD" H 7400 2550 50  0001 C CNN
 F 3 "~" H 7400 2550 50  0001 C CNN
 	1    7400 2550
@@
 F 0 "D6" V 7446 1470 50  0000 R CNN
 F 1 "D" V 7355 1470 50  0000 R CNN
-F 2 "kbd:D3_TH" H 7400 1550 50  0001 C CNN
+F 2 "kbd:D3_TH_SMD" H 7400 1550 50  0001 C CNN
 F 3 "~" H 7400 1550 50  0001 C CNN
 	1    7400 1550

Commit message: nkns1 rev.0.2
* Change row0-row5 port.
* Add rotary encoder.
Parts:
- removed SW26: SW_PUSH, kbd:CherryMX_MidHeight_Hotswap, symbol kbd:SW_PUSH
- added SW35: Rotary_Encoder_Switch, Rotary_Encoder:RotaryEncoder_Alps_EC12E-Switch_Vertical_H20mm, symbol Device:Rotary_Encoder_Switch
Connections:
- net GND: now also SW35.C
- net col6: now also SW35.S1
- net row0: now also U1.19 (F5/A2); no longer U1.18 (F6/A1)
- net row1: now also U1.18 (F6/A1); no longer U1.17 (F7/A0)
- net row2: now also U1.17 (F7/A0); no longer U1.16 (B1/15)
- net row3: now also U1.16 (B1/15); no longer U1.15 (B3/14)
- net row4: now also U1.15 (B3/14); no longer U1.14 (B2/16)
- net re2: now reaches U1.13 (B6/10)
- net re2: now also SW35.B
- net RE_SW: now reaches D25.2 (A)
- net RE_SW: now also SW35.S2
- new net re1: SW35.A, U1.14 (B2/16)
- no-connect marks 5 -> 3
Other:
- moved on the sheet: J1, J2
Changed lines of the file:
@@
 encoding utf-8
 Sheet 1 1
-Title "Ki-1 (nkns1)"
-Date "2020-11-03"
-Rev "0.1"
+Title "Ki-1-r0.2 (nkns1)"
+Date "2021-01-24"
+Rev "0.2"
 Comp "nekomimist.org"
 Comment1 ""
@@
 Wire Wire Line
 	9100 5050 9100 5500
-Wire Wire Line
-	7950 4450 7950 5500
-Connection ~ 7950 4450
-Wire Wire Line
-	7950 4000 7950 4450
 Connection ~ 8550 5950
 Wire Wire Line
@@
 $EndComp
 $Comp
-L Device:D D25
-U 1 1 5FA2D436
-P 8550 4600
-F 0 "D25" V 8596 4520 50  0000 R CNN
-F 1 "D" V 8505 4520 50  0000 R CNN
-F 2 "kbd:D3_TH_SMD" H 8550 4600 50  0001 C CNN
-F 3 "~" H 8550 4600 50  0001 C CNN
-	1    8550 4600
-	0    -1   -1   0
-$EndComp
-$Comp
 L Device:D D24
 U 1 1 5FA2D268
@@
 F 3 "" H 8250 5500 50  0000 C CNN
 	1    8250 5500
-	1    0    0    -1
-$EndComp
-$Comp
-L kbd:SW_PUSH SW26
-U 1 1 5FA269EB
-P 8250 4450
-F 0 "SW26" H 8250 4705 50  0000 C CNN
-F 1 "SW_PUSH" H 8250 4614 50  0000 C CNN
-F 2 "kbd:CherryMX_MidHeight_Hotswap" H 8250 4450 50  0001 C CNN
-F 3 "" H 8250 4450 50  0000 C CNN
-	1    8250 4450
 	1    0    0    -1
 $EndComp
@@
 Wire Wire Line
 	10050 3750 9800 3750
+Text GLabel 10200 2200 2    50   Input ~ 0
+row0
 Text GLabel 10200 2300 2    50   Input ~ 0
-row0
+row1
 Text GLabel 10200 2400 2    50   Input ~ 0
-row1
+row2
 Text GLabel 10200 2500 2    50   Input ~ 0
-row2
+row3
 Text GLabel 10200 2600 2    50   Input ~ 0
-row3
-Text GLabel 10200 2700 2    50   Input ~ 0
 row4
 Text GLabel 8800 2100 0    50   Input ~ 0
@@
 Text GLabel 8800 2800 0    50   Input ~ 0
 col7
-NoConn ~ 10200 2100
-NoConn ~ 10200 2200
 $Comp
 L power:GND #PWR09
 U 1 1 5FB57CD6
-P 2800 7100
-F 0 "#PWR09" H 2800 6850 50  0001 C CNN
-F 1 "GND" H 2805 6927 50  0000 C CNN
-F 2 "" H 2800 7100 50  0001 C CNN
-F 3 "" H 2800 7100 50  0001 C CNN
-	1    2800 7100
+P 1450 7100
+F 0 "#PWR09" H 1450 6850 50  0001 C CNN
+F 1 "GND" H 1455 6927 50  0000 C CNN
+F 2 "" H 1450 7100 50  0001 C CNN
+F 3 "" H 1450 7100 50  0001 C CNN
+	1    1450 7100
 	1    0    0    -1
 $EndComp
@@
 L power:VCC #PWR07
 U 1 1 5FB58F19
-P 2800 6750
-F 0 "#PWR07" H 2800 6600 50  0001 C CNN
-F 1 "VCC" H 2815 6923 50  0000 C CNN
-F 2 "" H 2800 6750 50  0001 C CNN
-F 3 "" H 2800 6750 50  0001 C CNN
-	1    2800 6750
-	1    0    0    -1
-$EndComp
-Wire Wire Line
-	2550 6875 2800 6875
+P 1450 6750
+F 0 "#PWR07" H 1450 6600 50  0001 C CNN
+F 1 "VCC" H 1465 6923 50  0000 C CNN
+F 2 "" H 1450 6750 50  0001 C CNN
+F 3 "" H 1450 6750 50  0001 C CNN
+	1    1450 6750
+	1    0    0    -1
+$EndComp
+Wire Wire Line
+	1200 6875 1450 6875
 $Comp
 L kbd:MJ-4PP-9 J1
 U 1 1 5FB56881
-P 2350 6900
-F 0 "J1" H 2381 7176 50  0000 C CNN
-F 1 "MJ-4PP-9" H 2381 7085 50  0000 C CNN
-F 2 "kbd:MJ-4PP-9" H 2625 7075 50  0001 C CNN
-F 3 "~" H 2625 7075 50  0001 C CNN
-	1    2350 6900
-	1    0    0    -1
-$EndComp
-Wire Wire Line
-	2800 6750 2800 6875
-Wire Wire Line
-	2550 6925 2800 6925
-Wire Wire Line
-	2800 6925 2800 7100
-NoConn ~ 2550 6825
-Text GLabel 2900 6975 2    50   Input ~ 0
+P 1000 6900
+F 0 "J1" H 1031 7176 50  0000 C CNN
+F 1 "MJ-4PP-9" H 1031 7085 50  0000 C CNN
+F 2 "kbd:MJ-4PP-9" H 1275 7075 50  0001 C CNN
+F 3 "~" H 1275 7075 50  0001 C CNN
+	1    1000 6900
+	1    0    0    -1
+$EndComp
+Wire Wire Line
+	1450 6750 1450 6875
+Wire Wire Line
+	1200 6925 1450 6925
+Wire Wire Line
+	1450 6925 1450 7100
+NoConn ~ 1200 6825
+Text GLabel 1550 6975 2    50   Input ~ 0
 data
 Wire Wire Line
-	2550 6975 2900 6975
+	1200 6975 1550 6975
 $Comp
 L power:VCC #PWR08
 U 1 1 5FA25C6F
-P 4500 6750
-F 0 "#PWR08" H 4500 6600 50  0001 C CNN
-F 1 "VCC" H 4515 6923 50  0000 C CNN
-F 2 "" H 4500 6750 50  0001 C CNN
-F 3 "" H 4500 6750 50  0001 C CNN
-	1    4500 6750
+P 3150 6750
+F 0 "#PWR08" H 3150 6600 50  0001 C CNN
+F 1 "VCC" H 3165 6923 50  0000 C CNN
+F 2 "" H 3150 6750 50  0001 C CNN
+F 3 "" H 3150 6750 50  0001 C CNN
+	1    3150 6750
 	1    0    0    -1
 $EndComp
@@
 L power:GND #PWR010
 U 1 1 5FA263D7
-P 4500 7100
-F 0 "#PWR010" H 4500 6850 50  0001 C CNN
-F 1 "GND" H 4505 6927 50  0000 C CNN
-F 2 "" H 4500 7100 50  0001 C CNN
-F 3 "" H 4500 7100 50  0001 C CNN
-	1    4500 7100
+P 3150 7100
+F 0 "#PWR010" H 3150 6850 50  0001 C CNN
+F 1 "GND" H 3155 6927 50  0000 C CNN
+F 2 "" H 3150 7100 50  0001 C CNN
+F 3 "" H 3150 7100 50  0001 C CNN
+	1    3150 7100
 	1    0    0    -1
 $EndComp
@@
 data
 NoConn ~ 10200 1700
-Text GLabel 4500 6950 2    50   Input ~ 0
+Text GLabel 3150 6950 2    50   Input ~ 0
 led
-NoConn ~ 10200 2800
-Wire Wire Line
-	4150 6950 4500 6950
-Wire Wire Line
-	4150 7050 4500 7050
-Wire Wire Line
-	4500 7050 4500 7100
-Wire Wire Line
-	4150 6850 4500 6850
-Wire Wire Line
-	4500 6850 4500 6750
+Wire Wire Line
+	2800 6950 3150 6950
+Wire Wire Line
+	2800 7050 3150 7050
+Wire Wire Line
+	3150 7050 3150 7100
+Wire Wire Line
+	2800 6850 3150 6850
+Wire Wire Line
+	3150 6850 3150 6750
 $Comp
 L Connector_Generic:Conn_01x03 J2
 U 1 1 5FAA66D7
-P 3950 6950
-F 0 "J2" H 3868 6625 50  0000 C CNN
-F 1 "SERIAL_LED" H 3868 6716 50  0000 C CNN
-F 2 "kbd:StripLED_rev" H 3950 6950 50  0001 C CNN
-F 3 "~" H 3950 6950 50  0001 C CNN
-	1    3950 6950
+P 2600 6950
+F 0 "J2" H 2518 6625 50  0000 C CNN
+F 1 "SERIAL_LED" H 2518 6716 50  0000 C CNN
+F 2 "kbd:StripLED_rev" H 2600 6950 50  0001 C CNN
+F 3 "~" H 2600 6950 50  0001 C CNN
+	1    2600 6950
 	-1   0    0    -1
 $EndComp
+Text GLabel 10200 2700 2    50   Input ~ 0
+re1
+$Comp
+L Device:Rotary_Encoder_Switch SW35
+U 1 1 601117CF
+P 4750 7000
+F 0 "SW35" H 4750 7367 50  0000 C CNN
+F 1 "Rotary_Encoder_Switch" H 4750 7276 50  0000 C CNN
+F 2 "Rotary_Encoder:RotaryEncoder_Alps_EC12E-Switch_Vertical_H20mm" H 4600 7160 50  0001 C CNN
+F 3 "~" H 4750 7260 50  0001 C CNN
+	1    4750 7000
+	1    0    0    -1
+$EndComp
+Text GLabel 4450 6900 0    50   Input ~ 0
+re1
+Text GLabel 4450 7100 0    50   Input ~ 0
+re2
+$Comp
+L power:GND #PWR0101
+U 1 1 601A180B
+P 4100 7150
+F 0 "#PWR0101" H 4100 6900 50  0001 C CNN
+F 1 "GND" H 4105 6977 50  0000 C CNN
+F 2 "" H 4100 7150 50  0001 C CNN
+F 3 "" H 4100 7150 50  0001 C CNN
+	1    4100 7150
+	1    0    0    -1
+$EndComp
+Wire Wire Line
+	4100 7150 4100 7000
+Wire Wire Line
+	4100 7000 4450 7000
+Text GLabel 8400 4400 0    50   Input ~ 0
+RE_SW
+Text GLabel 5050 6900 2    50   Input ~ 0
+col6
+Text GLabel 5050 7100 2    50   Input ~ 0
+RE_SW
+Text GLabel 10200 2800 2    50   Input ~ 0
+re2
+$Comp
+L Device:D D25
+U 1 1 5FA2D436
+P 8550 4600
+F 0 "D25" V 8596 4520 50  0000 R CNN
+F 1 "D" V 8505 4520 50  0000 R CNN
+F 2 "kbd:D3_TH_SMD" H 8550 4600 50  0001 C CNN
+F 3 "~" H 8550 4600 50  0001 C CNN
+	1    8550 4600
+	0    -1   -1   0
+$EndComp
+Wire Wire Line
+	7950 4000 7950 5500
+Wire Wire Line
+	8400 4400 8550 4400
+Wire Wire Line
+	8550 4400 8550 4450
+NoConn ~ 10200 2100
 $EndSCHEMATC
